File: Hardware/entrenador.sch (EAGLE design)
At the start: 59 parts, among them U1 DRV8833

Commit message: FALTA PONER LA SERIGRAFIA  .Arreglados todos los issues del circuito salvo determinar por que los pines meten ruido.
Parts:
- added C10, C13, C15, C16: 100n, adafruit:C-USC0805
- added U$10: SN74LVC2G04SOT23-6, frizzy:SN74LVC2G04SOT23-6
- C11, C12, C9: device SparkFun-Passives:CAP0603-CAP -> rcl:C-EUC0805
Connections:
- new net PWMA_N: U$1.A, U$10.2Y
- new net PWMB_N: U$10.1Y, U$9.A
- net GND: now also C10.2, C13.2, C15.2, C16.2, U$10.GND
- net PB1: now also C10.1
- net PB2: now also C13.1
- net PB3: now also C15.1
- net PB4: now also C16.1
- net PWMA: now also U$10.2A; no longer U$1.A
- net PWMB: now also U$10.1A; no longer U$9.A
- net RGB_G: now also R13.2; no longer R12.2
- net RGB_R: now also R12.2; no longer R13.2
- net VCC: now also U$10.VCC
Other:
- moved on the sheet: C8, D5, S5, U$2

Commit message: me falto revisar una cosa del anterior commit, disculpas. curregido
Changed lines of the file:
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@@
 <segment>
 <pinref part="C12" gate="G$1" pin="2"/>
-<label x="441.96" y="124.46" size="1.778" layer="95"/>
+<wire x1="447.04" y1="129.54" x2="447.04" y2="127" width="0.1524" layer="91"/>
+<label x="444.5" y="124.46" size="1.778" layer="95"/>
 </segment>
 </net>
